Commit message: forkeed from my RRIS repo

File: mbot_description/models/mbot_xacro/mbot_base_gazebo.xacro (robot description, xacro)
@@ -144,6 +144,6 @@
             <material>Gazebo/Blue</material>
         </gazebo>
-        <wheel prefix="left"  reflect="-1"/>
-        <wheel prefix="right" reflect="1"/>
+        <wheel prefix="left"  reflect="1"/>
+        <wheel prefix="right" reflect="-1"/>
         <caster prefix="front" reflect="-1"/>
         <caster prefix="back"  reflect="1"/>
@@ -154,5 +154,5 @@
                 <rosDebugLevel>Debug</rosDebugLevel>
                 <publishWheelTF>true</publishWheelTF>
-		<publishOdomTF>true</publishOdomTF>
+		        <publishOdomTF>true</publishOdomTF>
                 <robotNamespace>/</robotNamespace>
                 <publishTf>1</publishTf>
@@ -160,5 +160,5 @@
                 <alwaysOn>true</alwaysOn>
                 <updateRate>100.0</updateRate>
-                <legacyMode>true</legacyMode>
+                <legacyMode>false</legacyMode>
                 <leftJoint>left_wheel_joint</leftJoint>
                 <rightJoint>right_wheel_joint</rightJoint>

File: mbot_description/models/mbot_xacro/mbot_base_realsense.xacro (robot description, xacro)
@@ -1,5 +1,5 @@
 <?xml version="1.0"?>
 <robot name="mbot" xmlns:xacro="http://www.ros.org/wiki/xacro">
-    <xacro:include filename="$(find realsense_gazebo_plugin)/urdf/realsense-RS200.macro.xacro" />
+    <xacro:include filename="$(find mbot_description)/models/sensors/RealSense_D435.xacro" />
     <!-- PROPERTY LIST -->
     <xacro:property name="M_PI" value="3.1415926"/>
@@ -148,6 +148,6 @@
             <material>Gazebo/Blue</material>
         </gazebo>
-        <wheel prefix="left"  reflect="-1"/>
-        <wheel prefix="right" reflect="1"/>
+        <wheel prefix="left"  reflect="1"/>
+        <wheel prefix="right" reflect="-1"/>
         <caster prefix="front" reflect="-1"/>
         <caster prefix="back"  reflect="1"/>
@@ -167,5 +167,5 @@
                 <alwaysOn>true</alwaysOn>
                 <updateRate>100.0</updateRate>
-                <legacyMode>true</legacyMode>
+                <legacyMode>false</legacyMode>
                 <leftJoint>left_wheel_joint</leftJoint>
                 <rightJoint>right_wheel_joint</rightJoint>

File: mbot_description/models/mbot_xacro/mbot_with_camera_gazebo.xacro (robot description, xacro)
@@ -1,6 +1,6 @@
 <?xml version="1.0"?>
 <robot name="arm" xmlns:xacro="http://www.ros.org/wiki/xacro">
-    <xacro:include filename="$(find mbot_description)/urdf/xacro/gazebo/mbot_base_gazebo.xacro" />
-    <xacro:include filename="$(find mbot_description)/urdf/xacro/sensors/camera_gazebo.xacro" />
+    <xacro:include filename="$(find mbot_description)/models/mbot_xacro/mbot_base_gazebo.xacro" />
+    <xacro:include filename="$(find mbot_description)/models/sensors/camera_gazebo.xacro" />
     <xacro:property name="camera_offset_x" value="0.17" />
     <xacro:property name="camera_offset_y" value="0" />

File: mbot_description/models/nuric/base.urdf.xacro (robot description, xacro)
@@ -4,9 +4,10 @@
        xmlns:interface="http://playerstage.sourceforge.net/gazebo/xmlschema/#interface"
        xmlns:xacro="http://www.ros.org/wiki/xacro">
-  <xacro:include filename="$(find mbot_description)/urdf/xacro/nuric/wheelchair.gazebo.xacro" />
-  <xacro:include filename="$(find mbot_description)/urdf/xacro/nuric/wheelchair.transmission.xacro" />
-  <xacro:include filename="$(find mbot_description)/urdf/xacro/nuric/wheelchair.constants.xacro" />
-  <xacro:include filename="$(find mbot_description)/urdf/xacro/nuric/wheelchair.kinect.xacro" />
-  <xacro:include filename="$(find mbot_description)/urdf/xacro/nuric/wheelchair.hokuyo.xacro" />
+  <xacro:include filename="$(find mbot_description)/models/nuric/wheelchair.gazebo.xacro" />
+  <xacro:include filename="$(find mbot_description)/models/nuric/wheelchair.transmission.xacro" />
+  <xacro:include filename="$(find mbot_description)/models/nuric/wheelchair.constants.xacro" />
+  <xacro:include filename="$(find mbot_description)/models/nuric/wheelchair.kinect.xacro" />
+  <xacro:include filename="$(find mbot_description)/models/nuric/wheelchair.hokuyo.xacro" />
+  <xacro:include filename="$(find mbot_description)/models/sensors/lidar_gazebo.xacro" />
   <xacro:property name="PI" value="3.1415926535897931" />
   <xacro:property name="front_wheel_radius" value="0.17" />
@@ -21,13 +22,22 @@
   <xacro:property name="kinecty" value="0.0" />
   <xacro:property name="kinectz" value="1.41" />
-  <wheelchair_kinect_single parent="base_link" roll="0.025" pitch="0.25" yaw="0.0" x="${kinectx}" y="${kinecty}" z="${kinectz}" />
-  <wheelchair_hokuyo parent="base_link" roll="${PI}" pitch="0.0" yaw=" 0.0" x="0.25" y="0.0" z="-0.1" />
+  <xacro:property name="base_offset" value="0.0" />
+  <wheelchair_kinect_single parent="base_link" roll="0.0" pitch="0.2" yaw="0.0" x="${kinectx + base_offset}" y="${kinecty}" z="${kinectz}" />
+  <!-- hokuyo lidar at the bottom -->
+  <wheelchair_hokuyo parent="base_link" roll="${PI}" pitch="-0.1" yaw="0.0" x="${0.25 + base_offset}" y="0.0" z="0.1" />
+  <!-- 360 lidar on the top -->
+  <xacro:rplidar prefix="laser"/>
+  <joint name="lidar_joint" type="fixed">
+      <origin xyz="${base_offset - 0.75} 0 1.5" rpy="0.005 0 0" />
+      <parent link="base_link"/>
+      <child link="laser_link"/>
+  </joint>
   <!-- Macro for front wheel only -->
   <xacro:macro name="front_wheel" params="suffix parent reflect" >
     <joint name="${parent}_${suffix}_front_wheel_joint" type="continuous">
       <axis xyz="0 1 0" />
-      <limit effort="100" velocity="100" />
+      <limit effort="1000" velocity="1000" />
       <dynamics damping="0.0" friction="0.05" />
-      <origin xyz="0 ${reflect*front_wheel_base_y} 0" rpy="0 0 0" />
+      <origin xyz="${base_offset} ${reflect*front_wheel_base_y} 0" rpy="0 0 0" />
       <parent link="${parent}_link" />
       <child link="${suffix}_front_wheel_link" />
@@ -132,4 +142,30 @@
     </joint>
     <link name="base_link" >
+      <visual>
+        <origin xyz="0 0 0" rpy="0 0 0" />
+        <geometry>
+          <box size="0.01 0.01 0.01" />
+        </geometry>
+      </visual>
+    </link>
+    <joint name="dummy_link_joint" type="fixed" >
+      <origin xyz="-0.25 0 0" rpy="0 0 0" />
+      <child link="dummy_link" />
+      <parent link="base_link" />
+    </joint>
+    <link name="dummy_link" >
+      <visual>
+        <origin xyz="0 0 0" rpy="0 0 0" />
+        <geometry>
+          <box size="0.01 0.01 0.01" />
+        </geometry>
+      </visual>
+    </link>
+    <joint name="base_link_joint" type="fixed" >
+      <origin xyz="${base_offset} 0 0" rpy="0 0 0" />
+      <child link="wheelchair_link" />
+      <parent link="base_link" />
+    </joint>
+    <link name="wheelchair_link" >
       <xacro:wheelchair_base_inertia />
       <visual>
@@ -145,61 +181,15 @@
       </collision>
     </link>
-    <xacro:front_wheel suffix="left" parent="base" reflect="1" />
-    <xacro:front_wheel suffix="right" parent="base" reflect="-1" />
+    <xacro:front_wheel suffix="left" parent="base" reflect="-1" />
+    <xacro:front_wheel suffix="right" parent="base" reflect="1" />
     <xacro:caster_set suffix="left" parent="base" reflect="1" >
-      <origin xyz="${caster_hub_base_x} ${caster_hub_base_y} ${caster_hub_base_z}"
+      <origin xyz="${caster_hub_base_x + base_offset} ${caster_hub_base_y} ${caster_hub_base_z}"
               rpy="0 0 0" />
     </xacro:caster_set>
     <xacro:caster_set suffix="right" parent="base" reflect="-1" >
-      <origin xyz="${caster_hub_base_x} ${-caster_hub_base_y} ${caster_hub_base_z}"
+      <origin xyz="${caster_hub_base_x + base_offset} ${-caster_hub_base_y} ${caster_hub_base_z}"
               rpy="0 0 ${PI}" />
     </xacro:caster_set>
     <xacro:wheelchair_base_gazebo diameter="${2*front_wheel_radius}" separation="${2*front_wheel_base_y}" />
   </xacro:macro>
-<!-- =============================================================================== -->
-  <!-- Original Testing Macro for front wheels only -->
-  <!-- <xacro:macro name="f_wheel" >
-    <joint name="wheel_joint" type="continuous">
-      <axis xyz="0 1 0" />
-      <limit effort="100" velocity="100" />
-      <dynamics damping="0.0" friction="0.05" />
-      <origin xyz="0 0 0" rpy="${M_PI} 0 0" />
-      <parent link="wheelchair_base_link" />
-      <child link="base_f_wheel_link" />
-    </joint>
-    <link name="base_f_wheel_link" >
-      <visual>
-        <geometry>
-          <mesh filename="package://nuric_wheelchair_model_02/meshes/wheel.dae" />
-        </geometry>
-      </visual>
-    </link>
-  </xacro:macro> -->
-  <!-- Original Testing Macro for wheelchair_base (includes front & caster wheels and wheelchair body) -->
-  <!-- <xacro:macro name="wheelchair_base" >
-    <link name="base_footprint" >
-      <visual>
-        <origin xyz="0 0 0" rpy="0 0 0" />
-        <geometry>
-          <box size="0.01 0.01 0.01" />
-        </geometry>
-      </visual>
-    </link>
-    <joint name="base_footprint_joint" type="fixed" >
-      <origin xyz="0 0 ${f_wheel_radius}" rpy="0 0 0" />
-      <child link="wheelchair_base_link" />
-      <parent link="base_footprint" />
-    </joint>
-    <link name="wheelchair_base_link" >
-      <visual>
-        <origin xyz="0 0 0" rpy="0 0 0" />
-        <geometry>
-          <box size="0.4 0.3 0.05" />
-        </geometry>
-      </visual>
-    </link>
-    <xacro:f_wheel >
-    </xacro:f_wheel>
-  </xacro:macro> -->
-<!-- =============================================================================== -->
 </robot>

File: mbot_description/models/nuric/wheelchair.constants.xacro (robot description, xacro)
@@ -11,5 +11,5 @@
    <xacro:macro name="caster_wheel_inertia" >
       <inertial>
-        <mass value="0.07" />
+        <mass value="0.010" />
         <origin xyz="0 0 0" />
         <inertia  ixx="0.001" ixy="0.0" ixz="0.0"
@@ -19,5 +19,5 @@
    <xacro:macro name="caster_hub_inertia" params="lr">
       <inertial>
-        <mass value="0.015" />
+        <mass value="1.815" />
         <origin xyz="${lr*-0.043126} 0.030993 0.053064" />
         <inertia  ixx="0.001" ixy="0.0" ixz="0.0"
@@ -27,5 +27,5 @@
    <xacro:macro name="wheelchair_base_inertia" >
       <inertial>
-        <mass value="5.0" />
+        <mass value="10.0" />
         <origin xyz="-0.15 0.000000 0.1" />
         <inertia  ixx="0.011469" ixy="0.0" ixz="0.005697"

File: mbot_description/models/nuric/wheelchair.hokuyo.xacro (robot description, xacro)
@@ -42,11 +42,11 @@
           <samples>640</samples>
           <resolution>1</resolution>
-          <min_angle>-2.26889</min_angle>
-          <max_angle>2.26889</max_angle>
+          <min_angle>-1.85</min_angle>
+          <max_angle>1.85</max_angle>
         </horizontal>
       </scan>
       <range>
         <min>0.08</min>
-        <max>10.0</max>
+        <max>20.0</max>
         <resolution>0.01</resolution>
       </range>
@@ -61,5 +61,5 @@
       <alwaysOn>true</alwaysOn>
       <updateRate>20</updateRate>
-      <topicName>scan</topicName>
+      <topicName>/hokuyo/scan</topicName>
       <interface:laser name="gazebo_ros_laser_iface" />
       <frameName>laser_joint</frameName>

File: mbot_description/models/nuric/wheelchair.kinect.xacro (robot description, xacro)
@@ -137,8 +137,8 @@
       <visualize>true</visualize>
       <camera>
-        <horizontal_fov>1.047</horizontal_fov>
+        <horizontal_fov>2.047</horizontal_fov>
         <image>
-            <width>640</width>
-            <height>480</height>
+            <width>1280</width>
+            <height>720</height>
             <format>R8G8B8</format>
         </image>
@@ -147,5 +147,5 @@
         <clip>
             <near>0.1</near>
-            <far>6</far>
+            <far>20</far>
         </clip>
       </camera>
@@ -175,4 +175,40 @@
     </sensor>
   </gazebo>
+  <!-- <gazebo reference="camera_link">
+    <sensor type="camera" name="camera_color">
+      <always_on>true</always_on>
+      <visualize>true</visualize>
+      <update_rate>30</update_rate>
+      <camera>
+        <horizontal_fov>1.211</horizontal_fov>
+        <image>
+            <width>1920</width>
+            <height>1080</height>
+            <format>RGB_INT8</format>
+        </image>
+        <clip>
+            <near>0.1</near>
+            <far>20</far>
+        </clip>
+      </camera>
+    </sensor>
+    <sensor type="depth" name="camera_depth">
+      <always_on>true</always_on>
+      <visualize>false</visualize>
+      <update_rate>90</update_rate>
+      <camera>
+        <horizontal_fov>1.487</horizontal_fov>
+        <image>
+            <width>1280</width>
+            <height>720</height>
+            <format>R8G8B8</format>
+        </image>
+        <clip>
+            <near>0.1</near>
+            <far>20</far>
+        </clip>
+      </camera>
+    </sensor>
+  </gazebo> -->
 </xacro:macro>
 </robot>

File: mbot_description/models/nuric/wheelchair.urdf.xacro (robot description, xacro)
@@ -5,5 +5,5 @@
        xmlns:interface="http://playerstage.sourceforge.net/gazebo/xmlschema/#interface"
        xmlns:xacro="http://www.ros.org/wiki/xacro" >
-  <xacro:include filename="$(find mbot_description)/urdf/xacro/nuric/base.urdf.xacro" />
+  <xacro:include filename="$(find mbot_description)/models/nuric/base.urdf.xacro" />
   <xacro:wheelchair_base />
 </robot>

File: mbot_description/models/sensors/camera_gazebo.xacro (robot description, xacro)
@@ -51,5 +51,5 @@
                     <alwaysOn>true</alwaysOn>
                     <updateRate>0.0</updateRate>
-                    <cameraName>/camera</cameraName>
+                    <cameraName>/camera/rgb</cameraName>
                     <imageTopicName>image_raw</imageTopicName>
                     <cameraInfoTopicName>camera_info</cameraInfoTopicName>

File: mbot_description/models/sensors/lidar_gazebo.xacro (robot description, xacro)
@@ -38,11 +38,11 @@
                         <samples>360</samples>
                         <resolution>1.0</resolution>
-                        <min_angle>-3.142</min_angle>
-                        <max_angle>3.142</max_angle>
+                        <min_angle>-3.1415926</min_angle>
+                        <max_angle>3.124088224</max_angle>
                       </horizontal>
                     </scan>
                     <range>
                       <min>0.10</min>
-                      <max>15.0</max>
+                      <max>20.0</max>
                       <resolution>0.01</resolution>
                     </range>

Commit message: forked from my RRIS repo

File: mbot_description/models/mbot_xacro/mbot_base_gazebo.xacro (robot description, xacro)
@@ -119,4 +119,15 @@
         <gazebo reference="base_footprint">
             <turnGravityOff>false</turnGravityOff>
+            <sensor name="bumper_sensor" type="contact">
+            <always_on>true</always_on>
+            <update_rate>30</update_rate>
+            <contact>
+                <collision>base_footprint_fixed_joint_lump__base_link_collision</collision>
+            </contact>
+            <plugin name="bumper_plugin" filename="libgazebo_ros_bumper.so">
+                <bumperTopicName>mbot_base_collision</bumperTopicName>
+                <frameName>base_footprint</frameName>
+            </plugin>
+            </sensor>
         </gazebo>
         <joint name="base_footprint_joint" type="fixed">

File: mbot_description/models/nuric/base.urdf.xacro (robot description, xacro)
@@ -9,5 +9,4 @@
   <xacro:include filename="$(find mbot_description)/models/nuric/wheelchair.kinect.xacro" />
   <xacro:include filename="$(find mbot_description)/models/nuric/wheelchair.hokuyo.xacro" />
-  <xacro:include filename="$(find mbot_description)/models/sensors/lidar_gazebo.xacro" />
   <xacro:property name="PI" value="3.1415926535897931" />
   <xacro:property name="front_wheel_radius" value="0.17" />
@@ -22,15 +21,6 @@
   <xacro:property name="kinecty" value="0.0" />
   <xacro:property name="kinectz" value="1.41" />
-  <xacro:property name="base_offset" value="0.0" />
-  <wheelchair_kinect_single parent="base_link" roll="0.0" pitch="0.2" yaw="0.0" x="${kinectx + base_offset}" y="${kinecty}" z="${kinectz}" />
-  <!-- hokuyo lidar at the bottom -->
-  <wheelchair_hokuyo parent="base_link" roll="${PI}" pitch="-0.1" yaw="0.0" x="${0.25 + base_offset}" y="0.0" z="0.1" />
-  <!-- 360 lidar on the top -->
-  <xacro:rplidar prefix="laser"/>
-  <joint name="lidar_joint" type="fixed">
-      <origin xyz="${base_offset - 0.75} 0 1.5" rpy="0.005 0 0" />
-      <parent link="base_link"/>
-      <child link="laser_link"/>
-  </joint>
+  <wheelchair_kinect_single parent="base_link" roll="0.0" pitch="0.2" yaw="0.0" x="${kinectx}" y="${kinecty}" z="${kinectz}" />
+  <wheelchair_hokuyo parent="base_link" roll="${PI}" pitch="-0.1" yaw="0.0" x="0.25" y="0.0" z="0.1" />
   <!-- Macro for front wheel only -->
   <xacro:macro name="front_wheel" params="suffix parent reflect" >
@@ -39,5 +29,5 @@
       <limit effort="1000" velocity="1000" />
       <dynamics damping="0.0" friction="0.05" />
-      <origin xyz="${base_offset} ${reflect*front_wheel_base_y} 0" rpy="0 0 0" />
+      <origin xyz="0 ${reflect*front_wheel_base_y} 0" rpy="0 0 0" />
       <parent link="${parent}_link" />
       <child link="${suffix}_front_wheel_link" />
@@ -136,4 +126,20 @@
       </visual>
     </link>
+    <gazebo reference="base_footprint">
+        <turnGravityOff>false</turnGravityOff>
+        <sensor name="bumper_sensor" type="contact">
+        <always_on>true</always_on>
+        <update_rate>30</update_rate>
+        <contact>
+            <collision>base_footprint_fixed_joint_lump__base_link_collision</collision>
+            <collision>base_footprint_fixed_joint_lump__camera_link_collision_1</collision>
+            <collision>base_footprint_fixed_joint_lump__laser_joint_collision_2</collision>
+        </contact>
+        <plugin name="bumper_plugin" filename="libgazebo_ros_bumper.so">
+            <bumperTopicName>mbot_base_collision</bumperTopicName>
+            <frameName>base_footprint</frameName>
+        </plugin>
+        </sensor>
+    </gazebo>
     <joint name="base_footprint_joint" type="fixed" >
       <origin xyz="0 0 ${front_wheel_radius}" rpy="0 0 0" />
@@ -142,30 +148,4 @@
     </joint>
     <link name="base_link" >
-      <visual>
-        <origin xyz="0 0 0" rpy="0 0 0" />
-        <geometry>
-          <box size="0.01 0.01 0.01" />
-        </geometry>
-      </visual>
-    </link>
-    <joint name="dummy_link_joint" type="fixed" >
-      <origin xyz="-0.25 0 0" rpy="0 0 0" />
-      <child link="dummy_link" />
-      <parent link="base_link" />
-    </joint>
-    <link name="dummy_link" >
-      <visual>
-        <origin xyz="0 0 0" rpy="0 0 0" />
-        <geometry>
-          <box size="0.01 0.01 0.01" />
-        </geometry>
-      </visual>
-    </link>
-    <joint name="base_link_joint" type="fixed" >
-      <origin xyz="${base_offset} 0 0" rpy="0 0 0" />
-      <child link="wheelchair_link" />
-      <parent link="base_link" />
-    </joint>
-    <link name="wheelchair_link" >
       <xacro:wheelchair_base_inertia />
       <visual>
@@ -184,9 +164,9 @@
     <xacro:front_wheel suffix="right" parent="base" reflect="1" />
     <xacro:caster_set suffix="left" parent="base" reflect="1" >
-      <origin xyz="${caster_hub_base_x + base_offset} ${caster_hub_base_y} ${caster_hub_base_z}"
+      <origin xyz="${caster_hub_base_x} ${caster_hub_base_y} ${caster_hub_base_z}"
               rpy="0 0 0" />
     </xacro:caster_set>
     <xacro:caster_set suffix="right" parent="base" reflect="-1" >
-      <origin xyz="${caster_hub_base_x + base_offset} ${-caster_hub_base_y} ${caster_hub_base_z}"
+      <origin xyz="${caster_hub_base_x} ${-caster_hub_base_y} ${caster_hub_base_z}"
               rpy="0 0 ${PI}" />
     </xacro:caster_set>

File: mbot_description/models/nuric/wheelchair.hokuyo.xacro (robot description, xacro)
@@ -61,5 +61,5 @@
       <alwaysOn>true</alwaysOn>
       <updateRate>20</updateRate>
-      <topicName>/hokuyo/scan</topicName>
+      <topicName>scan</topicName>
       <interface:laser name="gazebo_ros_laser_iface" />
       <frameName>laser_joint</frameName>

File: mbot_description/models/sensors/lidar_gazebo.xacro (robot description, xacro)
@@ -29,5 +29,5 @@
         </gazebo>
         <gazebo reference="${prefix}_link">
-            <sensor type="ray" name="rplidar">
+            <sensor type="gpu_ray" name="rplidar">
                 <pose>0 0 0 0 0 0</pose>
                 <visualize>false</visualize>
@@ -36,6 +36,6 @@
                     <scan>
                       <horizontal>
-                        <samples>360</samples>
-                        <resolution>1.0</resolution>
+                        <samples>1440</samples>
+                        <resolution>0.25</resolution>
                         <min_angle>-3.1415926</min_angle>
                         <max_angle>3.124088224</max_angle>
@@ -53,5 +53,5 @@
                     </noise>
                 </ray>
-                <plugin name="gazebo_rplidar" filename="libgazebo_ros_laser.so">
+                <plugin name="gazebo_rplidar" filename="libgazebo_ros_gpu_laser.so">
                     <topicName>/scan</topicName>
                     <frameName>laser_link</frameName>
