Commit message: forked from my RRIS repo

File: mbot_description/models/mbot_xacro/mbot_base_gazebo.xacro (robot description, xacro)
@@ -4,5 +4,5 @@
     <xacro:property name="M_PI" value="3.1415926"/>
     <xacro:property name="base_mass"   value="20" />
-    <xacro:property name="base_radius" value="0.20"/>
+    <xacro:property name="base_radius" value="0.35"/>
     <xacro:property name="base_length" value="0.16"/>
     <xacro:property name="wheel_mass"   value="2" />

File: mbot_description/models/mbot_xacro/mbot_with_laser_camera_gazebo.xacro (robot description, xacro)
@@ -3,5 +3,6 @@
     <xacro:include filename="$(find mbot_description)/models/mbot_xacro/mbot_base_gazebo.xacro" />
     <xacro:include filename="$(find mbot_description)/models/sensors/lidar_gazebo.xacro" />
-    <xacro:include filename="$(find mbot_description)/models/sensors/camera_gazebo.xacro" />
+    <!-- <xacro:include filename="$(find mbot_description)/models/sensors/kinect_gazebo.xacro" /> -->
+    <xacro:include filename="$(find mbot_description)/models/nuric/wheelchair.kinect.xacro" />
     <xacro:property name="lidar_offset_x" value="0" />
     <xacro:property name="lidar_offset_y" value="0" />
@@ -9,11 +10,12 @@
     <xacro:property name="camera_offset_x" value="0" />
     <xacro:property name="camera_offset_y" value="0" />
-    <xacro:property name="camera_offset_z" value="0.15" />
-    <!-- Camera -->
-    <joint name="camera_joint" type="fixed">
+    <xacro:property name="camera_offset_z" value="1.5" />
+    <!-- kinect -->
+    <!-- <joint name="camera_joint" type="fixed">
         <origin xyz="${camera_offset_x} ${camera_offset_y} ${camera_offset_z}" rpy="0 0 0" />
         <parent link="base_link"/>
         <child link="camera_link"/>
-    </joint>
+    </joint> -->
+    <wheelchair_kinect_single parent="base_link" roll="0.0" pitch="0.2" yaw="0.0" x="${camera_offset_x}" y="${camera_offset_y}" z="${camera_offset_z}" />
     <!-- lidar -->
     <joint name="lidar_joint" type="fixed">
@@ -23,5 +25,5 @@
     </joint>
     <xacro:rplidar prefix="laser"/>
-    <xacro:usb_camera prefix="camera"/>
+    <!-- <xacro:kinect_camera prefix="camera"/> -->
     <mbot_base_gazebo/>
 </robot>

File: mbot_description/models/nuric/base.urdf.xacro (robot description, xacro)
@@ -173,3 +173,49 @@
     <xacro:wheelchair_base_gazebo diameter="${2*front_wheel_radius}" separation="${2*front_wheel_base_y}" />
   </xacro:macro>
+<!-- =============================================================================== -->
+  <!-- Original Testing Macro for front wheels only -->
+  <!-- <xacro:macro name="f_wheel" >
+    <joint name="wheel_joint" type="continuous">
+      <axis xyz="0 1 0" />
+      <limit effort="100" velocity="100" />
+      <dynamics damping="0.0" friction="0.05" />
+      <origin xyz="0 0 0" rpy="${M_PI} 0 0" />
+      <parent link="wheelchair_base_link" />
+      <child link="base_f_wheel_link" />
+    </joint>
+    <link name="base_f_wheel_link" >
+      <visual>
+        <geometry>
+          <mesh filename="package://nuric_wheelchair_model_02/meshes/wheel.dae" />
+        </geometry>
+      </visual>
+    </link>
+  </xacro:macro> -->
+  <!-- Original Testing Macro for wheelchair_base (includes front & caster wheels and wheelchair body) -->
+  <!-- <xacro:macro name="wheelchair_base" >
+    <link name="base_footprint" >
+      <visual>
+        <origin xyz="0 0 0" rpy="0 0 0" />
+        <geometry>
+          <box size="0.01 0.01 0.01" />
+        </geometry>
+      </visual>
+    </link>
+    <joint name="base_footprint_joint" type="fixed" >
+      <origin xyz="0 0 ${f_wheel_radius}" rpy="0 0 0" />
+      <child link="wheelchair_base_link" />
+      <parent link="base_footprint" />
+    </joint>
+    <link name="wheelchair_base_link" >
+      <visual>
+        <origin xyz="0 0 0" rpy="0 0 0" />
+        <geometry>
+          <box size="0.4 0.3 0.05" />
+        </geometry>
+      </visual>
+    </link>
+    <xacro:f_wheel >
+    </xacro:f_wheel>
+  </xacro:macro> -->
+<!-- =============================================================================== -->
 </robot>

File: mbot_description/models/sensors/camera_gazebo.xacro (robot description, xacro)
@@ -51,5 +51,5 @@
                     <alwaysOn>true</alwaysOn>
                     <updateRate>0.0</updateRate>
-                    <cameraName>/camera/rgb</cameraName>
+                    <cameraName>/camera</cameraName>
                     <imageTopicName>image_raw</imageTopicName>
                     <cameraInfoTopicName>camera_info</cameraInfoTopicName>

Commit message: forked from my RRIS repo

File: mbot_description/models/mbot_xacro/mbot_base_gazebo.xacro (robot description, xacro)
@@ -63,5 +63,5 @@
                 </geometry>
             </collision>
-            <cylinder_inertial_matrix  m="${wheel_mass}" r="${wheel_radius}" h="${wheel_length}" />
+            <xacro:cylinder_inertial_matrix  m="${wheel_mass}" r="${wheel_radius}" h="${wheel_length}" />
         </link>
         <gazebo reference="${prefix}_wheel_link">
@@ -102,5 +102,5 @@
                 </geometry>
             </collision>
-            <sphere_inertial_matrix  m="${caster_mass}" r="${caster_radius}" />
+            <xacro:sphere_inertial_matrix  m="${caster_mass}" r="${caster_radius}" />
         </link>
         <gazebo reference="${prefix}_caster_link">
@@ -150,13 +150,47 @@
                 </geometry>
             </collision>
-            <cylinder_inertial_matrix  m="${base_mass}" r="${base_radius}" h="${base_length}" />
+            <xacro:cylinder_inertial_matrix  m="${base_mass}" r="${base_radius}" h="${base_length}" />
         </link>
         <gazebo reference="base_link">
             <material>Gazebo/Blue</material>
         </gazebo>
-        <wheel prefix="left"  reflect="1"/>
-        <wheel prefix="right" reflect="-1"/>
-        <caster prefix="front" reflect="-1"/>
-        <caster prefix="back"  reflect="1"/>
+        <joint name="marker_joint" type="fixed">
+            <origin xyz="0 0.15 0.75" rpy="0 0 0" />
+            <parent link="base_link"/>
+            <child link="marker_link" />
+        </joint>
+        <link name="marker_link">
+            <visual>
+                <origin xyz=" 0 0 0" rpy="0 0 0" />
+                <geometry>
+                    <cylinder length="1.1" radius="0.02"/>
+                </geometry>
+                <!-- <material name="yellow" /> -->
+            </visual>
+        </link>
+        <gazebo reference="marker_link">
+            <material>Gazebo/Black</material>
+        </gazebo>
+        <joint name="marker_joint2" type="fixed">
+            <origin xyz="0 -0.15 0.75" rpy="0 0 0" />
+            <parent link="base_link"/>
+            <child link="marker_link2" />
+        </joint>
+        <link name="marker_link2">
+            <visual>
+                <origin xyz=" 0 0 0" rpy="0 0 0" />
+                <geometry>
+                    <cylinder length="1.1" radius="0.02"/>
+                </geometry>
+                <!-- <material name="yellow" /> -->
+            </visual>
+        </link>
+        <gazebo reference="marker_link2">
+            <material>Gazebo/Black</material>
+        </gazebo>
+        <xacro:wheel prefix="left"  reflect="1"/>
+        <xacro:wheel prefix="right" reflect="-1"/>
+        <xacro:caster prefix="front" reflect="-1"/>
+        <xacro:caster prefix="back"  reflect="1"/>
         <!-- controller -->
         <gazebo>
@@ -164,8 +198,8 @@
                     filename="libgazebo_ros_diff_drive.so">
                 <rosDebugLevel>Debug</rosDebugLevel>
-                <publishWheelTF>true</publishWheelTF>
+                <publishWheelTF>false</publishWheelTF>
 		        <publishOdomTF>true</publishOdomTF>
                 <robotNamespace>/</robotNamespace>
-                <publishTf>1</publishTf>
+                <publishTf>true</publishTf>
                 <publishWheelJointState>true</publishWheelJointState>
                 <alwaysOn>true</alwaysOn>
@@ -176,5 +210,5 @@
                 <wheelSeparation>${wheel_joint_y*2}</wheelSeparation>
                 <wheelDiameter>${2*wheel_radius}</wheelDiameter>
-                <broadcastTF>1</broadcastTF>
+                <broadcastTF>true</broadcastTF>
                 <wheelTorque>30</wheelTorque>
                 <wheelAcceleration>1.8</wheelAcceleration>

File: mbot_description/models/mbot_xacro/mbot_box_gazebo.xacro (robot description, xacro)
@@ -73,5 +73,5 @@
                 </geometry>
             </collision>
-            <cylinder_inertial_matrix  m="${wheel_mass}" r="${wheel_radius}" h="${wheel_length}" />
+            <xacro:cylinder_inertial_matrix  m="${wheel_mass}" r="${wheel_radius}" h="${wheel_length}" />
         </link>
         <gazebo reference="${prefix}_wheel_link">
@@ -112,5 +112,5 @@
                 </geometry>
             </collision>
-            <sphere_inertial_matrix  m="${caster_mass}" r="${caster_radius}" />
+            <xacro:sphere_inertial_matrix  m="${caster_mass}" r="${caster_radius}" />
         </link>
         <gazebo reference="${prefix}_caster_link">
@@ -129,4 +129,15 @@
         <gazebo reference="base_footprint">
             <turnGravityOff>false</turnGravityOff>
+            <sensor name="bumper_sensor" type="contact">
+            <always_on>true</always_on>
+            <update_rate>30</update_rate>
+            <contact>
+                <collision>base_footprint_fixed_joint_lump__base_link_collision</collision>
+            </contact>
+            <plugin name="bumper_plugin" filename="libgazebo_ros_bumper.so">
+                <bumperTopicName>mbot_base_collision</bumperTopicName>
+                <frameName>base_footprint</frameName>
+            </plugin>
+            </sensor>
         </gazebo>
         <joint name="base_footprint_joint" type="fixed">
@@ -165,13 +176,47 @@
                 </geometry>
             </collision>
-            <box_inertial_matrix  m="${base_mass}" h = "${base_height}" l = "${base_length}" w ="${base_width}" />
+            <xacro:box_inertial_matrix  m="${base_mass}" h = "${base_height}" l = "${base_length}" w ="${base_width}" />
         </link>
         <gazebo reference="base_link">
             <material>Gazebo/Blue</material>
         </gazebo>
-        <wheel prefix="left"  reflect="1"/>
-        <wheel prefix="right" reflect="-1"/>
-        <caster prefix="front" reflect="-1"/>
-        <caster prefix="back"  reflect="1"/>
+        <joint name="marker_joint" type="fixed">
+            <origin xyz="0 0.06 0.70" rpy="0 0 0" />
+            <parent link="base_link"/>
+            <child link="marker_link" />
+        </joint>
+        <link name="marker_link">
+            <visual>
+                <origin xyz=" 0 0 0" rpy="0 0 0" />
+                <geometry>
+                    <cylinder length="0.80" radius="0.01"/>
+                </geometry>
+                <!-- <material name="yellow" /> -->
+            </visual>
+        </link>
+        <gazebo reference="marker_link">
+            <material>Gazebo/Black</material>
+        </gazebo>
+        <joint name="marker_joint2" type="fixed">
+            <origin xyz="0 -0.06 0.70" rpy="0 0 0" />
+            <parent link="base_link"/>
+            <child link="marker_link2" />
+        </joint>
+        <link name="marker_link2">
+            <visual>
+                <origin xyz=" 0 0 0" rpy="0 0 0" />
+                <geometry>
+                    <cylinder length="0.80" radius="0.01"/>
+                </geometry>
+                <!-- <material name="yellow" /> -->
+            </visual>
+        </link>
+        <gazebo reference="marker_link2">
+            <material>Gazebo/Black</material>
+        </gazebo>
+        <xacro:wheel prefix="left"  reflect="1"/>
+        <xacro:wheel prefix="right" reflect="-1"/>
+        <xacro:caster prefix="front" reflect="-1"/>
+        <xacro:caster prefix="back"  reflect="1"/>
         <!-- controller -->
         <gazebo>
@@ -179,5 +224,5 @@
                     filename="libgazebo_ros_diff_drive.so">
                 <rosDebugLevel>Debug</rosDebugLevel>
-                <publishWheelTF>true</publishWheelTF>
+                <publishWheelTF>false</publishWheelTF>
 		        <publishOdomTF>true</publishOdomTF>
                 <robotNamespace>/</robotNamespace>

File: mbot_description/models/mbot_xacro/mbot_with_laser_camera_gazebo.xacro (robot description, xacro)
@@ -8,5 +8,5 @@
     <xacro:property name="lidar_offset_y" value="0" />
     <xacro:property name="lidar_offset_z" value="0.105" />
-    <xacro:property name="camera_offset_x" value="0" />
+    <xacro:property name="camera_offset_x" value="-0.2" />
     <xacro:property name="camera_offset_y" value="0" />
     <xacro:property name="camera_offset_z" value="1.5" />
@@ -17,5 +17,5 @@
         <child link="camera_link"/>
     </joint> -->
-    <wheelchair_kinect_single parent="base_link" roll="0.0" pitch="0.2" yaw="0.0" x="${camera_offset_x}" y="${camera_offset_y}" z="${camera_offset_z}" />
+    <xacro:wheelchair_kinect_single parent="base_link" roll="0.0" pitch="0.2" yaw="0.0" x="${camera_offset_x}" y="${camera_offset_y}" z="${camera_offset_z}" />
     <!-- lidar -->
     <joint name="lidar_joint" type="fixed">
@@ -26,4 +26,4 @@
     <xacro:rplidar prefix="laser"/>
     <!-- <xacro:kinect_camera prefix="camera"/> -->
-    <mbot_base_gazebo/>
+    <xacro:mbot_base_gazebo/>
 </robot>

File: mbot_description/models/mbot_xacro/mbot_with_laser_gazebo.xacro (robot description, xacro)
@@ -13,4 +13,4 @@
     </joint>
     <xacro:rplidar prefix="laser"/>
-    <mbot_base_gazebo/>
+    <xacro:mbot_base_gazebo/>
 </robot>

File: mbot_description/models/mbot_xacro/mbox_with_laser_camera_gazebo.xacro (robot description, xacro)
@@ -7,7 +7,7 @@
     <xacro:property name="lidar_offset_y" value="0" />
     <xacro:property name="lidar_offset_z" value="0.105" />
-    <xacro:property name="camera_offset_x" value="0" />
+    <xacro:property name="camera_offset_x" value="-0.15" />
     <xacro:property name="camera_offset_y" value="0" />
-    <xacro:property name="camera_offset_z" value="0.15" />
+    <xacro:property name="camera_offset_z" value="1.2" />
     <!-- Camera -->
     <joint name="camera_joint" type="fixed">
@@ -24,4 +24,4 @@
     <xacro:rplidar prefix="laser"/>
     <xacro:usb_camera prefix="camera"/>
-    <mbot_base_gazebo/>
+    <xacro:mbot_base_gazebo/>
 </robot>

File: mbot_description/models/nuric/base.urdf.xacro (robot description, xacro)
@@ -21,6 +21,6 @@
   <xacro:property name="kinecty" value="0.0" />
   <xacro:property name="kinectz" value="1.41" />
-  <wheelchair_kinect_single parent="base_link" roll="0.0" pitch="0.2" yaw="0.0" x="${kinectx}" y="${kinecty}" z="${kinectz}" />
-  <wheelchair_hokuyo parent="base_link" roll="${PI}" pitch="-0.1" yaw="0.0" x="0.25" y="0.0" z="0.1" />
+  <xacro:wheelchair_kinect_single parent="base_link" roll="0.0" pitch="0.2" yaw="0.0" x="${kinectx}" y="${kinecty}" z="${kinectz}" />
+  <xacro:wheelchair_hokuyo parent="base_link" roll="${PI}" pitch="-0.1" yaw="0.0" x="0.25" y="0.0" z="0.1" />
   <!-- Macro for front wheel only -->
   <xacro:macro name="front_wheel" params="suffix parent reflect" >
@@ -130,5 +130,5 @@
         <sensor name="bumper_sensor" type="contact">
         <always_on>true</always_on>
-        <update_rate>30</update_rate>
+        <update_rate>10</update_rate>
         <contact>
             <collision>base_footprint_fixed_joint_lump__base_link_collision</collision>

File: mbot_description/models/nuric/wheelchair.kinect.xacro (robot description, xacro)
@@ -71,5 +71,5 @@
       <origin xyz="0.0 0.0 0.0" rpy="0 0 0" />
       <geometry>
-        <box size="0.0730 .2760 0.0720"/>
+        <box size="0.0 0.0 0.0"/>
       </geometry>
     </collision>

File: mbot_description/models/sensors/camera_gazebo.xacro (robot description, xacro)
@@ -32,5 +32,5 @@
                 <update_rate>30.0</update_rate>
                 <camera name="head">
-                    <horizontal_fov>1.3962634</horizontal_fov>
+                    <horizontal_fov>1.8962634</horizontal_fov>
                     <image>
                         <width>1280</width>
